File: layouts/default/default.kicad_pcb (KiCad board)
At the start: 2 copper layers, 8 parts

Commit message: Changes n stuff
Parts:
- removed R3, R4: 330Ω ±1% 100mW, UNI_ROYAL_0603WAF3300T5E:R0603
- added LED1: , Hubei_KENTO_Elec_KT_0603R:LED0603-RD, F.Cu at (-33.5, -40.8)
- added LED2: , Hubei_KENTO_Elec_KT_0603R:LED0603-RD, F.Cu at (-21.5, -40.7)
- added R5: 1kΩ ±1% 62.5mW, UNI_ROYAL_0402WGF1001TCE:R0402, F.Cu at (-33.5, -36.9)
- added R6: 1kΩ ±1% 62.5mW, UNI_ROYAL_0402WGF1001TCE:R0402, F.Cu at (-21.5, -36.9)
- Q1: moved to F.Cu
- R1, R2: value 47kΩ ±1% 100mW -> 100kΩ ±1% 100mW; footprint UNI_ROYAL_0603WAF4702T5E:R0603 -> UNI_ROYAL_0603WAF1003T5E:R0603
- moved R2 16.7 mm to (-29.5, -40.8), turned to -90 degrees
- moved R1 16.0 mm to (-25.5, -40.8), turned to -90 degrees
- moved C2 11.9 mm to (-25.5, -35.3), turned to 90 degrees
- moved C1 10.5 mm to (-29.5, -35.3), turned to 90 degrees
- moved Q2 10.1 mm to (-32.5, -30.5)
- moved Q1 6.95 mm to (-23.5, -30.5), turned to 0 degrees
Connections:
- net c1-cathode renamed c1-C
- net c2-cathode renamed c2-C
Routing:
- net VIN_PAD: track 0.00 -> 12.0 mm
- net footprint-cathode-0: track 0.00 -> 2.64 mm
- net footprint-cathode-1: track 0.00 -> 2.54 mm

Commit message: Wild stuff
Parts:
- moved Q2 17.0 mm to (-16.0, -26.4)
- moved Q1 14.7 mm to (-38.0, -27.9), turned to 180 degrees
- moved LED2 11.0 mm to (-10.5, -40.7)
- moved R6 11.0 mm to (-10.5, -36.9)
- moved R5 7.16 mm to (-40.5, -35.4)
- moved C1 6.50 mm to (-23.0, -35.3)
- moved C2 6.48 mm to (-29.5, -30.2)
- moved R1 3.00 mm to (-22.5, -40.8)
- moved LED1 2.50 mm to (-36.0, -40.8)
- moved R2 1.00 mm to (-30.5, -40.8)
Connections:
- C1 pad 1: c1-C -> GND
- C2 pad 1: c2-C -> GND
- Q1 pad 3: c2-C -> GND
- Q2 pad 3: c1-C -> GND
Routing:
- net VIN_PAD: track 12.0 -> 0.14 mm
- net footprint-cathode-0: track 2.64 -> 0.00 mm
- net footprint-cathode-1: track 2.54 -> 0.00 mm

Commit message: sdfadsf
Parts:
- R5, R6: value 1kΩ ±1% 62.5mW -> 10kΩ ±1% 62.5mW; footprint UNI_ROYAL_0402WGF1001TCE:R0402 -> UNI_ROYAL_0402WGF1002TCE:R0402
- moved R5 191.1 mm to (114.0, 77.0)
- moved R2 190.5 mm to (121.5, 74.0)
- moved Q1 190.4 mm to (117.5, 82.0)
- moved LED1 189.3 mm to (114.5, 74.0)
- moved C 188.9 mm to (126.0, 77.0), turned to -90 degrees
- moved R1 186.1 mm to (125.5, 72.0)
- moved R6 182.8 mm to (132.0, 77.6)
- moved LED2 181.6 mm to (129.9, 74.5)
- moved Q2 179.5 mm to (125.5, 84.0), turned to 180 degrees
- moved C1 178.9 mm to (117.0, 76.0), turned to -90 degrees
- renumbered C2 to C
Connections:
- C pad 1: GND -> B
- C pad 2: c2-B -> led2-power-GND
- C1 pad 1: GND -> B
- C1 pad 2: c1-B -> led1-power-GND
- Q1 pad 1: c1-B -> B
- Q1 pad 2: GND -> v5-GND
- Q1 pad 3: GND -> led1-power-GND
- Q2 pad 1: c2-B -> B
- Q2 pad 2: GND -> v5-GND
- Q2 pad 3: GND -> led2-power-GND
- R1 pad 2: c1-B -> B
- R2 pad 2: c2-B -> B
- R5 pad 2: GND -> led1-power-GND
- R6 pad 2: GND -> led2-power-GND
Routing:
- net VIN_PAD: track 0.14 -> 17.5 mm
- net B: track 0.00 -> 9.69 mm
- net led2-power-GND: track 0.00 -> 6.64 mm
- net led1-power-GND: track 0.00 -> 3.30 mm
- net footprint-cathode-1: track 0.00 -> 2.88 mm
- net footprint-cathode-0: track 0.00 -> 1.98 mm

Commit message: init
Parts:
- removed C: 10µF ±10% 10V X5R, Samsung_Electro_Mechanics_CL10A106KP8NNNC:C0603
- removed R5, R6: 10kΩ ±1% 62.5mW, UNI_ROYAL_0402WGF1002TCE:R0402
- added C2: 10µF ±10% 10V X5R, Samsung_Electro_Mechanics_CL10A106KP8NNNC:C0603, F.Cu at (0.00, -10.0)
- added R3: 100kΩ ±1% 100mW, UNI_ROYAL_0603WAF1003T5E:R0603, F.Cu at (0.00, -40.0)
- added R4: 100kΩ ±1% 100mW, UNI_ROYAL_0603WAF1003T5E:R0603, F.Cu at (0.00, -50.0)
- R1, R2: value 100kΩ ±1% 100mW -> 10kΩ ±1% 62.5mW; footprint UNI_ROYAL_0603WAF1003T5E:R0603 -> UNI_ROYAL_0402WGF1002TCE:R0402
- moved Q2 169.5 mm to (0.00, -30.0), turned to 0 degrees
- moved Q1 155.6 mm to (0.00, -20.0), turned to 0 degrees
- moved C1 139.5 mm to (0.00, 0.00), turned to 0 degrees
- moved R1 136.1 mm to (10.0, 0.00), turned to 180 degrees
- moved LED1 126.0 mm to (12.5, 0.00), turned to 0 degrees
- moved LED2 122.6 mm to (32.5, 0.00), turned to 0 degrees
- moved R2 117.7 mm to (30.0, 0.00), turned to 180 degrees
Connections:
- net v5-GND renamed GND_PAD
- C1 pad 1: B -> led1.low
- C1 pad 2: led1-power-GND -> r1.unnamed[1]
- Q1 pad 1: B -> r2.unnamed[1]
- Q1 pad 3: led1-power-GND -> led1.low
- Q2 pad 1: B -> r1.unnamed[1]
- Q2 pad 3: led2-power-GND -> led2.low
- R1 pad 1: VIN_PAD -> footprint-cathode-0
- R1 pad 2: B -> led1.low
- R2 pad 1: VIN_PAD -> footprint-cathode-1
- R2 pad 2: B -> led2.low
Routing:
- net VIN_PAD: track 17.5 -> 0.00 mm
- net B: track 9.69 -> 0.00 mm
- net led2-power-GND: track 6.64 -> 0.00 mm
- net led1-power-GND: track 3.30 -> 0.00 mm
- net footprint-cathode-1: track 2.88 -> 1.27 mm
- net footprint-cathode-0: track 1.98 -> 1.27 mm

Commit message: messy
Parts:
- moved R4 212.6 mm to (177.0, 67.7)
- moved R3 208.7 mm to (177.0, 70.5)
- moved Q2 206.7 mm to (184.0, 64.2)
- moved Q1 206.3 mm to (184.0, 73.2)
- moved C2 196.3 mm to (180.5, 67.2)
- moved C1 193.7 mm to (180.5, 70.2)
- moved R1 184.8 mm to (179.7, 73.2), turned to 0 degrees
- moved LED1 180.3 mm to (177.2, 73.2), turned to 180 degrees
- moved R2 162.9 mm to (179.7, 64.2), turned to 0 degrees
- moved LED2 158.3 mm to (177.2, 64.2), turned to 180 degrees
Routing:
- net GND_PAD: track 0.00 -> 21.6 mm, vias 0 -> 2
- net r2.unnamed[1]: track 0.00 -> 12.0 mm, vias 0 -> 2
- net r1.unnamed[1]: track 0.00 -> 11.1 mm
- net VIN_PAD: track 0.00 -> 9.12 mm
- net led2.low: track 0.00 -> 6.01 mm
- net led1.low: track 0.00 -> 6.01 mm
- added copper zone on B.Cu, net GND_PAD
- added copper zone on F.Cu, net GND_PAD
Other:
- board outline added: 26 x 27.5 mm

Commit message: progreesa
Parts:
- added U1: , AMASS_XT30PW_F20_G_Y:CONN-TH_XT30PW-F-1, F.Cu at (162.8, 97.0)
- C1, C2: value 10µF ±10% 10V X5R -> (none); footprint Samsung_Electro_Mechanics_CL10A106KP8NNNC:C0603 -> Honor_Elec_RVT1V101M0607:CAP-SMD_BD6.3-L6.6-W6.6-FD
- R4: value 100kΩ ±1% 100mW -> 10kΩ ±1% 100mW; footprint UNI_ROYAL_0603WAF1003T5E:R0603 -> UNI_ROYAL_0603WAF1002T5E:R0603
- moved LED2 37.4 mm to (195.3, 97.0), turned to 0 degrees
- moved R2 35.3 mm to (192.8, 97.0), turned to 180 degrees
- moved R4 32.3 mm to (207.8, 77.8)
- moved R1 24.7 mm to (172.8, 97.0), turned to 180 degrees
- moved LED1 23.8 mm to (175.3, 97.0), turned to 0 degrees
- moved R3 22.0 mm to (197.8, 77.8)
- moved Q1 21.5 mm to (162.8, 77.0)
- moved Q2 21.4 mm to (162.8, 67.0)
- moved C2 12.8 mm to (187.8, 77.8)
- moved C1 7.99 mm to (177.8, 77.8)
Connections:
- net r1.unnamed[1] renamed r1.cathode
- net r2.unnamed[1] renamed r2.cathode
Routing:
- net GND_PAD: track 21.6 -> 0.00 mm, vias 2 -> 0
- net r2.cathode: track 12.0 -> 0.00 mm, vias 2 -> 0
- net r1.cathode: track 11.1 -> 0.00 mm
- net VIN_PAD: track 9.12 -> 0.00 mm
- net led2.low: track 6.01 -> 0.00 mm
- net led1.low: track 6.01 -> 0.00 mm
- removed copper zone on B.Cu, net GND_PAD
- removed copper zone on F.Cu, net GND_PAD
Other:
- board size 26 x 27.5 mm -> 174.5 x 101.5 mm
